Commit message: Use Xacro properties

File: grounds_bot_workspace/description_package/urdf/GroundsBot.urdf.xacro (robot description, xacro)
@@ -1,4 +1,8 @@
 <?xml version="1.0"?>
 <robot name="GroundsBot" xmlns:xacro="http://www.ros.org/wiki/xacro">
+  <!-- Xacro properties -->
+  <xacro:property name="width" value="3.2"/>
+  <xacro:property name="height" value="1.5"/>
+  <xacro:property name="length" value="3.6"/>
   <!-- Colors -->
   <material name="grey">
@@ -16,5 +20,5 @@
       <origin xyz="0 0 0.75" rpy="0 0 0"/>
       <geometry>
-        <box size="3.0 2.0 1.5"/>
+        <box size="3.0 ${width - 1.2} ${height}"/>
       </geometry>
       <material name="grey"/>
@@ -25,5 +29,5 @@
       <origin xyz="0.8 0 0.25" rpy="0 0 0"/>
       <geometry>
-        <box size="1.6 3.2 0.5"/>
+        <box size="1.6 ${width} ${height / 3}"/>
       </geometry>
       <material name="grey"/>
@@ -32,5 +36,5 @@
   <link name="left_wheel_link">
     <visual>
-      <origin xyz="0 0 0" rpy="1.5708 0 0"/>
+      <origin xyz="0 0 0" rpy="${pi/2} 0 0"/>
       <geometry>
         <cylinder radius="0.7" length="0.6"/>

Commit message: Added macro for a wheel

File: grounds_bot_workspace/description_package/urdf/GroundsBot.urdf.xacro (robot description, xacro)
@@ -15,4 +15,16 @@
     <color rgba="0.8 0.1 0.1 1.0"/>
   </material>
+  <!-- Xacro macros -->
+  <xacro:macro name="wheel" params="prefix">
+    <link name="${prefix}_wheel_link">
+      <visual>
+        <origin xyz="0 0 0" rpy="${pi/2} 0 0"/>
+        <geometry>
+          <cylinder radius="0.7" length="0.6"/>
+        </geometry>
+        <material name="black"/>
+      </visual>
+    </link>
+  </xacro:macro>
   <!-- Links -->
   <link name="base_link">
@@ -34,13 +46,5 @@
     </visual>
   </link>
-  <link name="left_wheel_link">
-    <visual>
-      <origin xyz="0 0 0" rpy="${pi/2} 0 0"/>
-      <geometry>
-        <cylinder radius="0.7" length="0.6"/>
-      </geometry>
-      <material name="black"/>
-    </visual>
-  </link>
+  <xacro:wheel prefix="left"/>
   <!-- Joints -->
   <joint name="base_cutting_unit_joint" type="fixed">

Commit message: Added front right wheel

File: grounds_bot_workspace/description_package/urdf/GroundsBot.urdf.xacro (robot description, xacro)
@@ -46,5 +46,6 @@
     </visual>
   </link>
-  <xacro:wheel prefix="left"/>
+  <xacro:wheel prefix="front_left"/>
+  <xacro:wheel prefix="front_right"/>
   <!-- Joints -->
   <joint name="base_cutting_unit_joint" type="fixed">
@@ -53,8 +54,14 @@
     <origin xyz="1.5 0 0" rpy="0 0 0"/>
   </joint>
-  <joint name="base_left_wheel_joint" type="continuous">
+  <joint name="base_front_left_wheel_joint" type="continuous">
     <parent link="base_link"/>
-    <child link="left_wheel_link"/>
+    <child link="front_left_wheel_link"/>
     <origin xyz="0.75 -1.3 0" rpy="0 0 0"/>
+    <axis xyz="0 1 0"/>
+  </joint>
+  <joint name="base_front_right_wheel_joint" type="continuous">
+    <parent link="base_link"/>
+    <child link="front_right_wheel_link"/>
+    <origin xyz="0.75 1.3 0" rpy="0 0 0"/>
     <axis xyz="0 1 0"/>
   </joint>

Commit message: Added rear tires

File: grounds_bot_workspace/description_package/urdf/GroundsBot.urdf.xacro (robot description, xacro)
@@ -47,5 +47,7 @@
   </link>
   <xacro:wheel prefix="front_left"/>
+  <xacro:wheel prefix="rear_left"/>
   <xacro:wheel prefix="front_right"/>
+  <xacro:wheel prefix="rear_right"/>
   <!-- Joints -->
   <joint name="base_cutting_unit_joint" type="fixed">
@@ -60,8 +62,20 @@
     <axis xyz="0 1 0"/>
   </joint>
+  <joint name="base_rear_left_wheel_joint" type="continuous">
+    <parent link="base_link"/>
+    <child link="rear_left_wheel_link"/>
+    <origin xyz="-0.75 -1.3 0" rpy="0 0 0"/>
+    <axis xyz="0 1 0"/>
+  </joint>
   <joint name="base_front_right_wheel_joint" type="continuous">
     <parent link="base_link"/>
     <child link="front_right_wheel_link"/>
     <origin xyz="0.75 1.3 0" rpy="0 0 0"/>
+    <axis xyz="0 1 0"/>
+  </joint>
+  <joint name="base_rear_right_wheel_joint" type="continuous">
+    <parent link="base_link"/>
+    <child link="rear_right_wheel_link"/>
+    <origin xyz="-0.75 1.3 0" rpy="0 0 0"/>
     <axis xyz="0 1 0"/>
   </joint>

Commit message: Improved xacro properties

File: grounds_bot_workspace/description_package/urdf/GroundsBot.urdf.xacro (robot description, xacro)
@@ -2,7 +2,9 @@
 <robot name="GroundsBot" xmlns:xacro="http://www.ros.org/wiki/xacro">
   <!-- Xacro properties -->
-  <xacro:property name="width" value="3.2"/>
+  <xacro:property name="width" value="3.0"/>
   <xacro:property name="height" value="1.5"/>
-  <xacro:property name="length" value="3.6"/>
+  <xacro:property name="length" value="4.5"/>
+  <xacro:property name="wheel_radius" value="0.7"/>
+  <xacro:property name="wheel_width" value="0.6"/>
   <!-- Colors -->
   <material name="grey">
@@ -21,5 +23,5 @@
         <origin xyz="0 0 0" rpy="${pi/2} 0 0"/>
         <geometry>
-          <cylinder radius="0.7" length="0.6"/>
+          <cylinder radius="${wheel_radius}" length="${wheel_width}"/>
         </geometry>
         <material name="black"/>
@@ -30,7 +32,7 @@
   <link name="base_link">
     <visual>
-      <origin xyz="0 0 0.75" rpy="0 0 0"/>
+      <origin xyz="0 0 ${height / 2}" rpy="0 0 0"/>
       <geometry>
-        <box size="3.0 ${width - 1.2} ${height}"/>
+        <box size="${(length / 3) * 2} ${width - (wheel_width * 2)} ${height}"/>
       </geometry>
       <material name="grey"/>
@@ -39,7 +41,7 @@
   <link name="cutting_unit_link">
     <visual>
-      <origin xyz="0.8 0 0.25" rpy="0 0 0"/>
+      <origin xyz="${length / 6} 0 ${height / 6}" rpy="0 0 0"/>
       <geometry>
-        <box size="1.6 ${width} ${height / 3}"/>
+        <box size="${length / 3} ${width} ${height / 3}"/>
       </geometry>
       <material name="grey"/>
@@ -54,10 +56,10 @@
     <parent link="base_link"/>
     <child link="cutting_unit_link"/>
-    <origin xyz="1.5 0 0" rpy="0 0 0"/>
+    <origin xyz="${length / 3} 0 0" rpy="0 0 0"/>
   </joint>
   <joint name="base_front_left_wheel_joint" type="continuous">
     <parent link="base_link"/>
     <child link="front_left_wheel_link"/>
-    <origin xyz="0.75 -1.3 0" rpy="0 0 0"/>
+    <origin xyz="${length / 6} ${(width - wheel_width) / -2} 0" rpy="0 0 0"/>
     <axis xyz="0 1 0"/>
   </joint>
@@ -65,5 +67,5 @@
     <parent link="base_link"/>
     <child link="rear_left_wheel_link"/>
-    <origin xyz="-0.75 -1.3 0" rpy="0 0 0"/>
+    <origin xyz="${length / -6} ${(width - wheel_width) / -2} 0" rpy="0 0 0"/>
     <axis xyz="0 1 0"/>
   </joint>
@@ -71,5 +73,5 @@
     <parent link="base_link"/>
     <child link="front_right_wheel_link"/>
-    <origin xyz="0.75 1.3 0" rpy="0 0 0"/>
+    <origin xyz="${length / 6} ${(width - wheel_width) / 2} 0" rpy="0 0 0"/>
     <axis xyz="0 1 0"/>
   </joint>
@@ -77,5 +79,5 @@
     <parent link="base_link"/>
     <child link="rear_right_wheel_link"/>
-    <origin xyz="-0.75 1.3 0" rpy="0 0 0"/>
+    <origin xyz="${length / -6} ${(width - wheel_width) / 2} 0" rpy="0 0 0"/>
     <axis xyz="0 1 0"/>
   </joint>

Commit message: Include the inertia tags

File: grounds_bot_workspace/description_package/urdf/GroundsBot.urdf.xacro (robot description, xacro)
@@ -1,4 +1,6 @@
 <?xml version="1.0"?>
 <robot name="GroundsBot" xmlns:xacro="http://www.ros.org/wiki/xacro">
+  <!-- Include other xacro files -->
+<xacro:include filename="$(find description_package)/urdf/inertia_properties.xacro" />
   <!-- Xacro properties -->
   <xacro:property name="width" value="3.0"/>
@@ -27,4 +29,6 @@
         <material name="black"/>
       </visual>
+      <xacro:cylinder_inertia m="0.25" r="${wheel_radius}" l="${wheel_width}"
+                              o_xyz="0 0 0" o_rpy="0 0 0"/>
     </link>
   </xacro:macro>
@@ -38,4 +42,6 @@
       <material name="grey"/>
     </visual>
+    <xacro:box_inertia m="3.0" x="${(length / 3) * 2}" y="${width - (wheel_width * 2)}" z="${height}"
+                       o_xyz="0 0 ${height / 2}" o_rpy="0 0 0"/>
   </link>
   <link name="cutting_unit_link">
@@ -47,4 +53,6 @@
       <material name="grey"/>
     </visual>
+    <xacro:box_inertia m="1.0" x="${length / 3}" y="${width}" z="${height / 3}"
+                       o_xyz="${length / 6} 0 ${height / 6}" o_rpy="0 0 0"/>
   </link>
   <xacro:wheel prefix="front_left"/>
@@ -83,13 +91,2 @@
   </joint>
 </robot>
-<!-- <collision>
-      <origin xyz="0 0 0" rpy="0 0 0"/>
-      <geometry>
-        <box size="2.0 1.2 0.4"/>
-      </geometry>
-    </collision>
-    <inertial>
-      <origin xyz="0 0 0" rpy="0 0 0"/>
-      <mass value="200.0"/>
-      <inertia ixx="16.0" iyy="66.7" izz="80.7" ixy="0" ixz="0" iyz="0"/>
-    </inertial> -->

File: grounds_bot_workspace/description_package/urdf/inertia_properties.xacro (robot description, xacro)
@@ -2,5 +2,5 @@
 <robot name="GroundsBot" xmlns:xacro="http://www.ros.org/wiki/xacro">
   <!-- Typical inertia for a box (parameters: mass, x-length, y-length, z-length, origin_xyz, origin_rpy) -->
-  <xacro:macro name="bos_inertia" params="m x y z o_xyz o_rpy">
+  <xacro:macro name="box_inertia" params="m x y z o_xyz o_rpy">
     <inertial>
       <mass value="${m}"/>
