Commit message: Corrected project structure

File: grounds_bot_workspace/src/description_package/urdf/GroundsBot.urdf.xacro (robot description, xacro)
@@ -29,4 +29,10 @@
         <material name="black"/>
       </visual>
+      <collision>
+        <geometry>
+          <cylinder radius="${wheel_radius}" length="${wheel_width}"/>
+        </geometry>
+        <origin xyz="" rpy=""/>
+      </collision>
       <xacro:cylinder_inertia m="0.25" r="${wheel_radius}" l="${wheel_width}"
                               o_xyz="0 0 0" o_rpy="0 0 0"/>
@@ -42,4 +48,10 @@
       <material name="grey"/>
     </visual>
+    <collision>
+      <geometry>
+        <box size="${(length / 3) * 2} ${width - (wheel_width * 2)} ${height}"/>
+      </geometry>
+      <origin xyz="" rpy=""/>
+    </collision>
     <xacro:box_inertia m="3.0" x="${(length / 3) * 2}" y="${width - (wheel_width * 2)}" z="${height}"
                        o_xyz="0 0 ${height / 2}" o_rpy="0 0 0"/>
@@ -53,4 +65,10 @@
       <material name="grey"/>
     </visual>
+    <collision>
+      <geometry>
+          <box size="${length / 3} ${width} ${height / 3}"/>
+      </geometry>
+      <origin xyz="" rpy=""/>
+    </collision>
     <xacro:box_inertia m="1.0" x="${length / 3}" y="${width}" z="${height / 3}"
                        o_xyz="${length / 6} 0 ${height / 6}" o_rpy="0 0 0"/>

Commit message: Completed collision tags

File: grounds_bot_workspace/src/description_package/urdf/GroundsBot.urdf.xacro (robot description, xacro)
@@ -33,8 +33,8 @@
           <cylinder radius="${wheel_radius}" length="${wheel_width}"/>
         </geometry>
-        <origin xyz="" rpy=""/>
+        <origin xyz="0 0 0" rpy="${pi/2} 0 0"/>
       </collision>
       <xacro:cylinder_inertia m="0.25" r="${wheel_radius}" l="${wheel_width}"
-                              o_xyz="0 0 0" o_rpy="0 0 0"/>
+                              o_xyz="0 0 0" o_rpy="${pi/2} 0 0"/>
     </link>
   </xacro:macro>
@@ -52,5 +52,5 @@
         <box size="${(length / 3) * 2} ${width - (wheel_width * 2)} ${height}"/>
       </geometry>
-      <origin xyz="" rpy=""/>
+      <origin xyz="0 0 ${height / 2}" rpy="0 0 0"/>
     </collision>
     <xacro:box_inertia m="3.0" x="${(length / 3) * 2}" y="${width - (wheel_width * 2)}" z="${height}"
@@ -69,5 +69,5 @@
           <box size="${length / 3} ${width} ${height / 3}"/>
       </geometry>
-      <origin xyz="" rpy=""/>
+      <origin xyz="${length / 6} 0 ${height / 6}" rpy="0 0 0"/>
     </collision>
     <xacro:box_inertia m="1.0" x="${length / 3}" y="${width}" z="${height / 3}"
