Commit message: Improvements using Xacro
Refactored differential drive configuration for clarity and structure.

File: grounds_bot_workspace/src/description_package/urdf/grounds_bot_gazebo.xacro (robot description, xacro)
@@ -1,5 +1,21 @@
 <?xml version="1.0"?>
 <robot xmlns:xacro="http://www.ros.org/wiki/xacro">
-  <!-- Differential drive for the front wheels -->
+  <!-- Basic differential drive -->
+  <xacro:macro name="differential_drive" params="left_joint right_joint">
+    <gazebo>
+      <plugin filename="gz-sim-diff-drive-system" name="gz::sim::systems::DiffDrive">
+        <left_joint>${left_joint}</left_joint>
+        <right_joint>${right_joint}</right_joint>
+        <frame_id>odom</frame_id>
+        <child_frame_id>base_footprint</child_frame_id>
+        <wheel_separation>1.8</wheel_separation>
+        <wheel_radius>0.6</wheel_radius>
+      </plugin>
+    </gazebo>
+  </xacro:macro>
+  <!-- Differential drives -->
+  <xacro:differential_drive left_joint="base_front_left_wheel_joint" right_joint="base_front_right_wheel_joint"/>
+  <xacro:differential_drive left_joint="base_rear_left_wheel_joint" right_joint="base_rear_right_wheel_joint"/>
+  <!-- Differential drive for the front wheels
   <gazebo>
     <plugin filename="gz-sim-diff-drive-system" name="gz::sim::systems::DiffDrive">
@@ -12,5 +28,5 @@
     </plugin>
   </gazebo>
-  <!-- Differential drive for the rear wheels -->
+  <!-- Differential drive for the rear wheels
   <gazebo>
     <plugin filename="gz-sim-diff-drive-system" name="gz::sim::systems::DiffDrive">
@@ -22,5 +38,5 @@
       <wheel_radius>0.6</wheel_radius>
     </plugin>
-  </gazebo>
+  </gazebo> -->
   <!-- Enable steering &c. -->
   <gazebo>

Commit message: Further Simplifications

File: grounds_bot_workspace/src/description_package/urdf/grounds_bot_gazebo.xacro (robot description, xacro)
@@ -1,42 +1,17 @@
 <?xml version="1.0"?>
 <robot xmlns:xacro="http://www.ros.org/wiki/xacro">
-  <!-- Basic differential drive -->
-  <xacro:macro name="differential_drive" params="left_joint right_joint">
-    <gazebo>
-      <plugin filename="gz-sim-diff-drive-system" name="gz::sim::systems::DiffDrive">
-        <left_joint>${left_joint}</left_joint>
-        <right_joint>${right_joint}</right_joint>
-        <frame_id>odom</frame_id>
-        <child_frame_id>base_footprint</child_frame_id>
-        <wheel_separation>1.8</wheel_separation>
-        <wheel_radius>0.6</wheel_radius>
-      </plugin>
-    </gazebo>
-  </xacro:macro>
-  <!-- Differential drives -->
-  <xacro:differential_drive left_joint="base_front_left_wheel_joint" right_joint="base_front_right_wheel_joint"/>
-  <xacro:differential_drive left_joint="base_rear_left_wheel_joint" right_joint="base_rear_right_wheel_joint"/>
-  <!-- Differential drive for the front wheels
+  <!-- Differential drive for each wheel -->
   <gazebo>
     <plugin filename="gz-sim-diff-drive-system" name="gz::sim::systems::DiffDrive">
       <left_joint>base_front_left_wheel_joint</left_joint>
+      <left_joint>base_rear_left_wheel_joint</left_joint>
       <right_joint>base_front_right_wheel_joint</right_joint>
-      <frame_id>odom</frame_id>
-      <child_frame_id>base_footprint</child_frame_id>
-      <wheel_separation>1.8</wheel_separation>
-      <wheel_radius>0.6</wheel_radius>
-    </plugin>
-  </gazebo>
-  <!-- Differential drive for the rear wheels
-  <gazebo>
-    <plugin filename="gz-sim-diff-drive-system" name="gz::sim::systems::DiffDrive">
-      <left_joint>base_rear_left_wheel_joint</left_joint>
       <right_joint>base_rear_right_wheel_joint</right_joint>
       <frame_id>odom</frame_id>
       <child_frame_id>base_footprint</child_frame_id>
-      <wheel_separation>1.8</wheel_separation>
-      <wheel_radius>0.6</wheel_radius>
+      <wheel_separation>${width - wheel_width}</wheel_separation>
+      <wheel_radius>${wheel_radius}</wheel_radius>
     </plugin>
-  </gazebo> -->
+  </gazebo>
   <!-- Enable steering &c. -->
   <gazebo>
